File: electrical/kicad/filaSens-attiny84.kicad_pcb (KiCad board)
At the start: 2 copper layers, 50 x 20 mm, 26 parts, among them J1 OUTPUT, J2 OUTPUT, J3 ISP, U1 ATtiny84-20SSU, U2 AT24C02D-STUM-T, U3 SS49X

Commit message: * Removed DS2402, twas a silly choice for a board with the option of being an i2c slave  * Updated silkscreen for better readability  * Added DS2431 one wire eeprom to replace the i2c one  * Moved STATUS and FAULT pins around to better fit part placement  * Added an (optional) mounting point for a ceramic resonator, mostly in case of an attiny84 setup for an external clock source  * Added iBom files
Parts:
- removed R7, R8: 4k7, Resistor_SMD:R_0402_1005Metric_Pad0.72x0.64mm_HandSolder
- removed the REF** at (144.2, 103.8)
- added Y1: AEL ZTT MT 8Mhz, Connector_PinHeader_2.54mm:PinHeader_1x03_P2.54mm_Vertical, F.Cu at (145.8, 112.7)
- U2: value AT24C02D-STUM-T -> DS2431; footprint Package_TO_SOT_SMD:SOT-23-5 -> Package_SO_J-Lead:TSOC-6_3.76x3.94mm_P1.27mm
- moved U1 2.90 mm to (143.3, 106.8)
- moved U2 1.19 mm to (150.7, 106.8), turned to 0 degrees
- moved J1 0.72 mm to (163.4, 98.5)
Connections:
- U1 pad 11: Net-(U1-Pad11) -> /MEM
- U1 pad 12: Net-(U1-Pad12) -> /FAULT
- U1 pad 13: /FAULT -> /STATUS
- U1 pad 2: /STATUS -> Net-(U1-Pad2)
- U2 pad 1: /SCL -> GND
- U2 pad 2: GND -> /MEM
- U2 pad 3: /SDA -> Net-(U2-Pad3)
- U2 pad 4: /+5v -> Net-(U2-Pad4)
- U2 pad 5: GND -> Net-(U2-Pad5)
Routing:
- net /+5v: track 84.4 -> 57.4 mm, vias 2 -> 0
- net /SCL: track 45.4 -> 30.6 mm
- net /SDA: track 42.3 -> 30.4 mm
- net /RESET: track 39.6 -> 29.9 mm, vias 1 -> 2
- net GND: track 10.3 -> 2.70 mm, vias 3 -> 2
- net /MEM: track 0.00 -> 7.23 mm, vias 0 -> 2
- net /STATUS: track 11.3 -> 5.42 mm
- net Net-(U1-Pad3): track 0.00 -> 5.39 mm
- net Net-(U1-Pad2): track 0.00 -> 3.43 mm
- net /PWM: track 11.4 -> 8.40 mm
- net /IN: track 9.24 -> 7.00 mm
- net /FAULT: track 42.9 -> 41.2 mm
- net /MISO: track 15.5 -> 13.8 mm
- net Net-(S1-Pad1): track 25.3 -> 24.1 mm
Other:
- board text added: "RST"
- board text added: "SCL/RX"
- board text added: "SDA/TX"
- board text added: "rev1 - Modified V0.2 Filament Diameter Sensor Licensed as Public Domain Designed by Thomas Sanladerer Modified by Mike "MiggyMan" Woods"
- board text removed: "RSET"
- board text removed: "SCL"
- board text removed: "SDA"
- board text removed: "rev1 - Modified Filament Diameter Sensor Licensed as Public Domain Designed by Thomas Sanladerer Modified by Mike "MiggyMan" Woods"

Commit message: * Split output headers into serial/i2c/analogue/power * Rearranged i2c/analouge/power headers to better fit horizontal pin headers * Made R5 throughole to make it easier to change and experiment with * Fixed reset button cockup * Change eeprom from i2c to one wire because having an i2c eeprom on an i2c slave device is kind of dumb
Parts:
- removed Y1: AEL ZTT MT 8Mhz, Connector_PinHeader_2.54mm:PinHeader_1x03_P2.54mm_Vertical
- added J4: OUT, Connector_PinHeader_2.54mm:PinHeader_1x03_P2.54mm_Vertical, F.Cu at (168.7, 109.9)
- added J5: SERIAL, Connector_PinHeader_2.54mm:PinHeader_1x03_P2.54mm_Vertical, F.Cu at (145.8, 112.4)
- added R7: 10k, Resistor_SMD:R_0402_1005Metric_Pad0.72x0.64mm_HandSolder, F.Cu at (149.4, 98.4)
- J1: value OUTPUT -> I2C; footprint Connector_PinHeader_2.54mm:PinHeader_1x06_P2.54mm_Vertical -> Connector_PinHeader_2.54mm:PinHeader_1x03_P2.54mm_Vertical
- J2: value OUTPUT -> POWER; footprint Connector_PinHeader_2.54mm:PinHeader_1x06_P2.54mm_Vertical -> Connector_PinHeader_2.54mm:PinHeader_1x02_P2.54mm_Vertical
- R5: footprint Resistor_SMD:R_0402_1005Metric_Pad0.72x0.64mm_HandSolder -> Resistor_THT:R_Axial_DIN0204_L3.6mm_D1.6mm_P2.54mm_Vertical
- moved J2 9.67 mm to (164.7, 106.3), turned to 180 degrees
- moved C2 6.66 mm to (158.2, 104.5), turned to 180 degrees
- moved J1 5.52 mm to (168.7, 100.1), turned to 270 degrees
- moved R5 1.99 mm to (141.2, 100.5)
Connections:
- J1 pad 1: /+5v -> GND
- J1 pad 2: GND -> /SCL
- J1 pad 3: /SCL -> /SDA
- J2 pad 1: /+5v -> GND
- J2 pad 2: GND -> /+5v
- S2 pad 2: /+5v -> GND
- U1 pad 2: Net-(U1-Pad2) -> /TX
- U1 pad 3: Net-(U1-Pad3) -> /RX
Routing:
- net /SDA: track 30.4 -> 22.1 mm
- net /FAULT: track 41.2 -> 33.3 mm
- net /SCL: track 30.6 -> 25.0 mm
- net Net-(U1-Pad3): track 5.39 -> 0.00 mm
- net /RESET: track 29.9 -> 33.6 mm
- net /OUT: track 30.3 -> 26.6 mm
- net /RX: track 0.00 -> 3.67 mm
- net Net-(S1-Pad1): track 24.1 -> 20.5 mm
- net Net-(U1-Pad2): track 3.43 -> 0.00 mm
- net /TX: track 0.00 -> 3.16 mm
- net /+5v: track 57.4 -> 54.3 mm, vias 0 -> 1
- net /IN: track 7.00 -> 5.21 mm
- net Net-(JP1-Pad1): track 1.98 -> 2.55 mm
Other:
- board text added: "RX"
- board text added: "SCL"
- board text added: "SDA"
- board text added: "TX"
- board text removed: "SCL/RX"
- board text removed: "SDA/TX"

Commit message: * Updated the block model for v0.3 board layout * Updated gerbers, bom and placement files
Other:
- board text added: "rev1 - Modified V0.3 Filament Diameter Sensor Licensed as Public Domain Designed by Thomas Sanladerer Modified by Mike "MiggyMan" Woods"
- board text removed: "rev1 - Modified V0.2 Filament Diameter Sensor Licensed as Public Domain Designed by Thomas Sanladerer Modified by Mike "MiggyMan" Woods"
